File: QuadMotorHAT.kicad_pcb (KiCad board)
At the start: 2 copper layers, 65 x 56 mm, 13 parts, among them J1 GPIO, J2 MPWR, J3 M3/GND/M4, J4 M1/GND/M2, U2 L293D, U3 L293D

Commit message: Improved PCB
Parts:
- added C1: 0.1uF, Capacitor_SMD:C_0805_2012Metric, F.Cu at (118.4, 83.0)
- added C3: 0.1uF, Capacitor_SMD:C_0805_2012Metric, F.Cu at (138.5, 83.0)
- added C4: 0.1uF, Capacitor_SMD:C_0805_2012Metric, F.Cu at (115.3, 61.3)
- added C5: 0.1uF, Capacitor_SMD:C_0805_2012Metric, F.Cu at (144.6, 59.9)
- D1: footprint LED_SMD:LED_0201_0603Metric -> LED_SMD:LED_0805_2012Metric
- R1: footprint Resistor_SMD:R_0201_0603Metric -> Resistor_SMD:R_0805_2012Metric
- moved R1 1.63 mm to (114.4, 56.1)
- moved D1 1.34 mm to (110.7, 56.1)
Routing:
- net GND: track 21.3 -> 0.00 mm, vias 0 -> 5
- net +5V: track 38.9 -> 58.8 mm
- net Net-(J2-Pin_2): track 87.9 -> 99.6 mm
- net Net-(J3-Pin_4): track 60.1 -> 66.3 mm
- net Net-(D1-A): track 3.88 -> 1.89 mm
Other:
- board text added: "GND"
- board text added: "PWR"
