File: QuadMotorHAT.kicad_sch (KiCad schematic)
At the start: 9 parts, among them J1 GPIO, J2 MPWR, J3 M3/GND/M4, J4 M1/GND/M2, U2 L293D, U3 L293D

Commit message: Improved PCB
Parts:
- added C1, C3, C4, C5: 0.1uF, Capacitor_SMD:C_0805_2012Metric, symbol Device:C
- D1: footprint LED_SMD:LED_0201_0603Metric -> LED_SMD:LED_0805_2012Metric
- R1: footprint Resistor_SMD:R_0201_0603Metric -> Resistor_SMD:R_0805_2012Metric
Connections:
- net +5V: now also C1.2, C4.2
- net GND: now also C1.1, C3.2, C4.1, C5.2
- net at C2.1, J2.2 (Pin_2), U2.8 (VCC2)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: now also C3.1, C5.1
